File: Hardware/openfanhub/fan_connector.kicad_sch (KiCad schematic)
At the start: 1 part, among them M9 Fan_4pin

Commit message: Update (not sure what)
Parts:
- renumbered M9 to M18
Changed lines of the file:
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@@
   (symbol (lib_id "power:GND") (at 76.2 92.71 0)
     (in_bom yes) (on_board yes)
-    (property "Reference" "#PWR083" (id 0) (at 76.2 99.06 0)
+    (property "Reference" "#PWR096" (id 0) (at 76.2 99.06 0)
       (effects (font (size 1.27 1.27)) hide)
     )
@@
   (symbol (lib_id "Motor:Fan_4pin") (at 76.2 85.09 0)
     (in_bom yes) (on_board yes)
-    (property "Reference" "M9" (id 0) (at 80.2132 82.6516 0)
+    (property "Reference" "M18" (id 0) (at 80.2132 82.6516 0)
       (effects (font (size 1.27 1.27)) (justify left))
     )

Commit message: update
Parts:
- renumbered M18 to M1
Connections:
- net GND: now also M1.4 (-); no longer M1.1 (-)
- net POWER_IN: now also M1.3 (+); no longer M1.2 (+)
- net PWM_IN: now also M1.1 (PWM); no longer M1.4 (PWM)
- net RPM_OUT: now also M1.2 (Tacho); no longer M1.3 (Tacho)
Changed lines of the file:
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@@
   (symbol (lib_id "Motor:Fan_4pin") (at 76.2 85.09 0)
     (in_bom yes) (on_board yes)
-    (property "Reference" "M18" (id 0) (at 80.2132 82.6516 0)
+    (property "Reference" "M1" (id 0) (at 80.2132 82.6516 0)
       (effects (font (size 1.27 1.27)) (justify left))
     )
